File: MeArmPiHat.kicad_pcb (KiCad board)
At the start: 2 copper layers, 65 x 56.5 mm, 26 parts, among them P1 CONN_02X03, P2 Raspberry_Pi_+_Conn, P3 CONN_01X02, P4 USB_OTG, P5 CONN_01X04, Q1 BSS138, U1 24C16, U2 PCF8591, U3 DMMT5401

Commit message: v1.4 of the Pi HAT
Parts:
- removed P3: CONN_01X02, Pin_Headers:Pin_Header_Straight_1x02
- added R10: 3.9k, Resistors_SMD:R_0603, B.Cu at (127.3, 81.5)
- added R9: 3.9k, Resistors_SMD:R_0603, B.Cu at (124.2, 81.5)
- ART2: footprint Custom:MEARM_LOGO -> Custom:MEARM_LOGO_NEW_LARGE
- D1: footprint LEDs:LED-RGB-5MM_Common_Cathode -> Custom:LED-RGB-5MM_Common_Cathode
- P4: footprint Custom:MOLEX_MICRO_USB_REVERSED -> Custom:AMPHENOL_MICRO_USB_REVERSED
- Q1: value BSS138 -> DMG2305
- R6, R7, R8: value R -> 250R
- moved ART2 25.0 mm to (149.1, 97.4)
- moved ART3 1.82 mm to (148.5, 91.9)
- moved U2 0.79 mm to (130.4, 88.4)
- moved P4 0.60 mm to (125.6, 124.5)
- moved Q1 0.47 mm to (123.0, 84.1)
Connections:
- P2 pad 10: Net-(P2-Pad10) -> (no net)
- P2 pad 12: Net-(P2-Pad12) -> (no net)
- P2 pad 13: Net-(P2-Pad13) -> (no net)
- P2 pad 16: Net-(P2-Pad16) -> (no net)
- P2 pad 18: Net-(P2-Pad18) -> (no net)
- P2 pad 21: Net-(P2-Pad21) -> (no net)
- P2 pad 22: Net-(P2-Pad22) -> (no net)
- P2 pad 32: Net-(P2-Pad32) -> (no net)
- P2 pad 33: Net-(P2-Pad33) -> (no net)
- P2 pad 35: Net-(P2-Pad35) -> (no net)
- P2 pad 36: Net-(P2-Pad36) -> (no net)
- P2 pad 40: Net-(P2-Pad40) -> (no net)
- P2 pad 8: Net-(P2-Pad8) -> (no net)
- P4 pad 2: Net-(P4-Pad2) -> (no net)
- P4 pad 3: Net-(P4-Pad3) -> (no net)
- P4 pad 4: Net-(P4-Pad4) -> (no net)
- R2 pad 1: Net-(P3-Pad2) -> Net-(P2-Pad37)
- U1 pad 7: Net-(P3-Pad2) -> Net-(P2-Pad37)
- U2 pad 11: Net-(U2-Pad11) -> (no net)
- U2 pad 15: Net-(U2-Pad15) -> (no net)
Routing:
- net Net-(P2-Pad37): track 0.00 -> 45.6 mm
- net Net-(P3-Pad2): track 34.6 -> 0.00 mm
- net GND: track 21.3 -> 31.9 mm
- net VSS: track 75.3 -> 69.3 mm
- net +3V3: track 160.0 -> 164.9 mm
- net /Joysticks/SCL: track 54.5 -> 57.0 mm
- net Net-(RV1-Pad2): track 7.59 -> 9.93 mm
- net /Joysticks/SDA: track 45.2 -> 46.9 mm
Other:
- board text added: "-"
- board text added: "MeArm Pi HAT v1.4 © 2017 Mime Industries Ltd"
- board text removed: "MeArm Pi HAT v1.1 © 2016 Mime Industries Ltd"
